Commit message: 11/10 Fix urdf

File: urdf/crane_x7_d435.urdf (robot description, URDF)
Before this commit: robot crane_x7, 24 links, 23 joints
Links:
- link camera_link: geometry collision mesh filename=package://crane_x7_description/meshes/visual/d435.obj; visual mesh filename=package://crane_x7_description/meshes/visual/d435.obj
- link crane_x7_gripper_base_link: geometry collision mesh filename=package://crane_x7_description/meshes/visual/wide_two_finge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 scale=1 1 1; visual mesh filename=package://crane_x7_description/meshes/visual/wide_two_finge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 scale=1 1 1
- link crane_x7_gripper_finger_a_link: geometry collision mesh filename=package://crane_x7_description/meshes/visual/wide_two_finge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 scale=1 1 1; visual mesh filename=package://crane_x7_description/meshes/visual/wide_two_finge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 scale=1 1 1
- link crane_x7_gripper_finger_b_link: geometry collision mesh filename=package://crane_x7_description/meshes/visual/wide_two_finge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 scale=1 1 1; visual mesh filename=package://crane_x7_description/meshes/visual/wide_two_finge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 scale=1 1 1
- link crane_x7_lower_arm_fixed_part_link: geometry collision mesh filename=package://crane_x7_description/meshes/visual/rotating_link_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 scale=1 1 1; visual mesh filename=package://crane_x7_description/meshes/visual/rotating_link_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 scale=1 1 1
- link crane_x7_lower_arm_revolute_part_link: geometry collision mesh filename=package://crane_x7_description/meshes/visual/rotating_link_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 scale=1 1 1; visual mesh filename=package://crane_x7_description/meshes/visual/rotating_link_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 scale=1 1 1
- link crane_x7_mounting_plate_link: geometry collision mesh filename=package://crane_x7_description/meshes/visual/mounting_plate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 scale=1 1 1; visual mesh filename=package://crane_x7_description/meshes/visual/mounting_plate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 scale=1 1 1
- link crane_x7_shoulder_fixed_part_link: geometry collision mesh filename=package://crane_x7_description/meshes/visual/base_fixed_par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 scale=1 1 1; visual mesh filename=package://crane_x7_description/meshes/visual/base_fixed_par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 scale=1 1 1
- link crane_x7_shoulder_revolute_part_link: geometry collision mesh filename=package://crane_x7_description/meshes/visual/base_revolute_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 scale=1 1 1; visual mesh filename=package://crane_x7_description/meshes/visual/base_revolute_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 scale=1 1 1
- link crane_x7_upper_arm_fixed_part_link: geometry collision mesh filename=package://crane_x7_description/meshes/visual/rotating_link_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 scale=1 1 1; visual mesh filename=package://crane_x7_description/meshes/visual/rotating_link_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 scale=1 1 1
- link crane_x7_upper_arm_revolute_part_link: geometry collision mesh filename=package://crane_x7_description/meshes/visual/rotating_link_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 scale=1 1 1; visual mesh filename=package://crane_x7_description/meshes/visual/rotating_link_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 scale=1 1 1
- link crane_x7_wrist_link: geometry collision mesh filename=package://crane_x7_description/meshes/visual/wrist.stl scale=1 1 1; visual mesh filename=package://crane_x7_description/meshes/visual/wrist.stl scale=1 1 1
