Commit message: 12/11 Fix urdf

File: urdf/crane_x7.urdf (robot description, URDF)
Before this commit: robot crane_x7, 22 links, 21 joints
Joints:
- joint crane_x7_lower_arm_fixed_part_joint: limit lower=-2.7401669256310974 upper=2.7401669256310974 effort=4.0 velocity=4.81710873 -> lower=0.0 upper=0.0 effort=4.0 velocity=4.81710873

File: urdf/crane_x7_d435.urdf (robot description, URDF)
Before this commit: robot crane_x7, 24 links, 23 joints
Joints:
- joint crane_x7_lower_arm_fixed_part_joint: limit lower=-2.7401669256310974 upper=2.7401669256310974 effort=4.0 velocity=4.81710873 -> lower=0.0 upper=0.0 effort=4.0 velocity=4.81710873

Commit message: 12/21 Fix urdf

File: urdf/crane_x7.urdf (robot description, URDF)
Before this commit: robot crane_x7, 22 links, 21 joints
Links:
- link crane_x7_gripper_base_link: geometry collision mesh filename=package://crane_x7_description/meshes/visual/wide_two_finge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 scale=1 1 1; visual mesh filename=package://crane_x7_description/meshes/collision/wide_two_fi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 scale=1 1 1
- link crane_x7_gripper_finger_a_link: geometry collision mesh filename=package://crane_x7_description/meshes/visual/wide_two_finge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 scale=1 1 1; visual mesh filename=package://crane_x7_description/meshes/collision/wide_two_fi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 scale=1 1 1
- link crane_x7_gripper_finger_b_link: geometry collision mesh filename=package://crane_x7_description/meshes/visual/wide_two_finge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 scale=1 1 1; visual mesh filename=package://crane_x7_description/meshes/collision/wide_two_fi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 scale=1 1 1

Commit message: 12/21 Fix urdf

File: urdf/crane_x7.urdf (robot description, URDF)
Before this commit: robot crane_x7, 22 links, 21 joints
Links:
- link crane_x7_gripper_base_link: geometry collision mesh filename=package://crane_x7_description/meshes/collision/wide_two_fi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 scale=1 1 1; visual mesh filename=package://crane_x7_description/meshes/visual/wide_two_finge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 scale=1 1 1
- link crane_x7_gripper_finger_a_link: geometry collision mesh filename=package://crane_x7_description/meshes/collision/wide_two_fi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 scale=1 1 1; visual mesh filename=package://crane_x7_description/meshes/visual/wide_two_finge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 scale=1 1 1
- link crane_x7_gripper_finger_b_link: geometry collision mesh filename=package://crane_x7_description/meshes/collision/wide_two_fi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 scale=1 1 1; visual mesh filename=package://crane_x7_description/meshes/visual/wide_two_finge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 scale=1 1 1
- link crane_x7_lower_arm_fixed_part_link: geometry collision mesh filename=package://crane_x7_description/meshes/collision/rotating_li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 scale=1 1 1; visual mesh filename=package://crane_x7_description/meshes/visual/rotating_link_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 scale=1 1 1
- link crane_x7_lower_arm_revolute_part_link: geometry collision mesh filename=package://crane_x7_description/meshes/collision/rotating_li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 scale=1 1 1; visual mesh filename=package://crane_x7_description/meshes/visual/rotating_link_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 scale=1 1 1
- link crane_x7_mounting_plate_link: geometry collision mesh filename=package://crane_x7_description/meshes/collision/mounting_pl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 scale=1 1 1; visual mesh filename=package://crane_x7_description/meshes/visual/mounting_plate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 scale=1 1 1
- link crane_x7_shoulder_fixed_part_link: geometry collision mesh filename=package://crane_x7_description/meshes/collision/base_fixed_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 scale=1 1 1; visual mesh filename=package://crane_x7_description/meshes/visual/base_fixed_par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 scale=1 1 1
- link crane_x7_upper_arm_fixed_part_link: geometry collision mesh filename=package://crane_x7_description/meshes/collision/rotating_li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 scale=1 1 1; visual mesh filename=package://crane_x7_description/meshes/visual/rotating_link_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 scale=1 1 1
- link crane_x7_upper_arm_revolute_part_link: geometry collision mesh filename=package://crane_x7_description/meshes/collision/rotating_li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 scale=1 1 1; visual mesh filename=package://crane_x7_description/meshes/visual/rotating_link_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 scale=1 1 1
- link crane_x7_wrist_link: geometry collision mesh filename=package://crane_x7_description/meshes/collision/wrist.stl scale=1 1 1; visual mesh filename=package://crane_x7_description/meshes/visual/wrist.stl scale=1 1 1
